File: MotorController/MotorController.kicad_sch (KiCad schematic)
At the start: 4 parts, among them U1 TMC2209_SILENTSTEPSTICK

Commit message: 2 Driver Design Done
Parts:
- removed R1, R2: R, symbol Device:R
- removed U1: TMC2209_SILENTSTEPSTICK, TMC2209_SILENTSTEPSTICK:MODULE_TMC2209_SILENTSTEPSTICK, symbol TMC2209_SILENTSTEPSTICK:TMC2209_SILENTSTEPSTICK
- added C1, C2: 470u, Capacitor_THT:CP_Radial_D6.3mm_P2.50mm, symbol Device:C
- added J1: Conn_01x02_Pin, Connector_PinSocket_2.54mm:PinSocket_1x02_P2.54mm_Vertical, symbol Connector:Conn_01x02_Pin
- added J2, J3: Conn_01x04_Pin, Connector_PinHeader_2.54mm:PinHeader_1x04_P2.54mm_Vertical, symbol Connector:Conn_01x04_Pin
- added J4, J5: Conn_01x01_Pin, Connector_PinSocket_2.54mm:PinSocket_1x01_P2.54mm_Vertical, symbol Connector:Conn_01x01_Pin
- added R12, R3: 1K, Resistor_THT:R_Axial_DIN0617_L17.0mm_D6.0mm_P5.08mm_Vertical, symbol Device:R
- added TP1: EN1, TestPoint:TestPoint_Pad_2.0x2.0mm, symbol Connector:TestPoint
- added TP2: EN2, TestPoint:TestPoint_Pad_2.0x2.0mm, symbol Connector:TestPoint
- added TP3: STEP1, TestPoint:TestPoint_Pad_2.0x2.0mm, symbol Connector:TestPoint
- added TP4: DIR1, TestPoint:TestPoint_Pad_2.0x2.0mm, symbol Connector:TestPoint
- added TP5: STEP2, TestPoint:TestPoint_Pad_2.0x2.0mm, symbol Connector:TestPoint
- added TP6: DIR2, TestPoint:TestPoint_Pad_2.0x2.0mm, symbol Connector:TestPoint
- added TP7: UART2, TestPoint:TestPoint_Pad_2.0x2.0mm, symbol Connector:TestPoint
- added TP8: UART1, TestPoint:TestPoint_Pad_2.0x2.0mm, symbol Connector:TestPoint
- added U3, U4: TMC2209_SILENTSTEPSTICK, TMC2209_SILENTSTEPSTICK:MODULE_TMC2209_SILENTSTEPSTICK, symbol TMC2209_SILENTSTEPSTICK:TMC2209_SILENTSTEPSTICK
Connections:
- net GND: now also U2.17 (GND), U2.2 (GND), C1.2, C2.2, J1.2 (Pin_2), J5.1 (Pin_1), U3.1 (GND), U3.7 (GND), U4.1 (GND), U4.7 (GND)
- net +5V: now reaches U2.1 (VIN)
- net +5V: now also C1.1, C2.1, J1.1 (Pin_1), J4.1 (Pin_1), U3.8 (VM), U4.8 (VM)
- net STEP1: now reaches U2.10 (GPIO32)
- net STEP1: now also TP3.1, U4.10 (STEP)
- net EN2: now reaches U2.13 (GPIO39)
- net EN2: now also TP2.1, U3.16 (~{EN})
- net EN1: now reaches U2.14 (GPIO36)
- net EN1: now also TP1.1, U4.16 (~{EN})
- net +3V3: now reaches U2.16 (3.3v)
- net +3V3: now also U3.2 (VIO), U4.2 (VIO)
- net UART2: now reaches U2.21 (GPIO16)
- net UART2: now also R12.2, TP7.1, U3.12 (UART)
- net at U2.22 (GPIO17): now also R12.1
- net UART1: now reaches U2.27 (GPIO3)
- net UART1: now also R3.2, TP8.1, U4.12 (UART)
- net at U2.28 (GPIO1): now also R3.1
- net DIR2: now reaches U2.7 (GPIO26)
- net DIR2: now also TP6.1, U3.9 (DIR)
- net STEP2: now reaches U2.8 (GPIO25)
- net STEP2: now also TP5.1, U3.10 (STEP)
- net DIR1: now reaches U2.9 (GPIO33)
- net DIR1: now also TP4.1, U4.9 (DIR)
- new net: J2.1 (Pin_1), U3.3 (M2A)
- new net: J2.2 (Pin_2), U3.4 (M1A)
- new net: J2.3 (Pin_3), U3.5 (M1B)
- new net: J2.4 (Pin_4), U3.6 (M2B)
- new net: J3.1 (Pin_1), U4.3 (M2A)
- new net: J3.2 (Pin_2), U4.4 (M1A)
- new net: J3.3 (Pin_3), U4.5 (M1B)
- new net: J3.4 (Pin_4), U4.6 (M2B)
- no-connect marks 6 -> 28
Other:
- note added: "Connectors"
- note added: "MCU"
- note added: "Motor Drivers"
- note removed: "TODO: Add Schottky on VM"
- note removed: "TODO: Check if EN is nEN or EN"
- note removed: "TODO: Verify UART Config"
- moved on the sheet: U2
